File: AL60.kicad_sch (KiCad schematic)
At the start: 177 parts, among them J1 USB_C_Receptacle_USB2.0, J2 JTAG_TC2030, SW1 Boot, U1 XC6206, U2 USBLC6-2SC6, U3 RP2040, U4 W25Q128JVS, Y1 12MHz

Commit message: Data lines and power routed
Parts:
- added D60: 1N4148, qw-footprints:CUSTOM D_SOD-123, symbol Device:D_Small
- added J3: DB JST, Connector_JST:JST_SH_SM04B-SRSS-TB_1x04-1MP_P1.00mm_Horizontal, symbol Connector:Conn_01x04_Male
- added MX60, MX62, MX66, MX78: MX_SW_solder, PCM_marbastlib-xp-alps:SW_Alps_MX_1.5u, symbol PCM_marbastlib-mx:MX_SW_solder
- added MX61, MX63, MX65, MX77, MX79, MX80, MX81, MX82, MX84: MX_SW_solder, PCM_marbastlib-xp-alps:SW_Alps_MX_1u, symbol PCM_marbastlib-mx:MX_SW_solder
- added MX83: MX_SW_solder, PCM_marbastlib-xp-alps:SW_Alps_MX_1.75u, symbol PCM_marbastlib-mx:MX_SW_solder
- S1: footprint PCM_marbastlib-mx:STAB_MX_P_6.25u -> PCM_marbastlib-mx:STAB_MX_6.25u
- S2: footprint PCM_marbastlib-mx:STAB_MX_P_7u -> PCM_marbastlib-mx:STAB_MX_7u
- S3: footprint PCM_marbastlib-mx:STAB_MX_P_2u -> PCM_marbastlib-mx:STAB_MX_2u
- S4, S7: footprint PCM_marbastlib-mx:STAB_MX_P_2.25u -> PCM_marbastlib-mx:STAB_MX_2.25u
- S5: footprint PCM_marbastlib-mx:STAB_MX_P_ISO -> PCM_marbastlib-mx:STAB_MX_ISO
- S6: footprint PCM_marbastlib-mx:STAB_MX_P_2.75u -> PCM_marbastlib-mx:STAB_MX_2.75u
Connections:
- net +5V: no longer U2.5 (VBUS)
- net D+: now also U2.1 (I/O1); no longer U2.6 (I/O1)
- net D-: now also U2.3 (I/O2); no longer U2.4 (I/O2)
- net DBUS+: now also U2.6 (I/O1), J3.3 (Pin_3); no longer U2.1 (I/O1)
- net DBUS-: now also U2.4 (I/O2), J3.2 (Pin_2); no longer U2.3 (I/O2)
- net GND: now also J3.4 (Pin_4)
- net at MX71.1: now also MX14.2, MX28.2, MX42.2, MX56.2, MX70.2, MX74.1, MX78.2, MX82.1
- net at MX71.2: now also D14.2 (A), MX14.1
- net at D58.2 (A), MX58.1: now also MX61.1
- net at MX16.2, MX2.2, MX30.2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: now also MX61.2
- net at D57.1 (K), D58.1 (K), D59.1 (K)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: now also D60.1 (K)
- net at D69.2 (A), MX69.1: now also MX77.1, MX81.2
- net at D54.2 (A), MX54.1: now also MX83.2
- net at MX10.2, MX24.2, MX38.2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: now also MX67.2, MX65.2
- net at D41.2 (A), MX41.1: now also MX73.1
- net at MX13.2, MX27.2, MX41.2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: now also MX73.2, MX76.1, MX77.2, MX81.1, MX84.1
- net at MX11.2, MX25.2, MX39.2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: now also MX68.2, MX66.2, MX79.2; no longer MX67.2
- net at MX12.2, MX26.2, MX40.2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: now also MX80.2, MX83.1; no longer MX68.2
- net at MX76.2: now also D55.2 (A), MX55.1, MX84.2
- net at MX22.2, MX36.2, MX50.2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: now also MX63.2
- net at MX75.1: now also D43.2 (A), MX43.1
- net at MX75.2: now also MX1.2, MX15.2, MX29.2, MX43.2, MX57.2, MX72.1, MX60.2
- net VCC: now reaches F1.1, J1.A4 (VBUS), J1.A9 (VBUS), J1.B4 (VBUS), J1.B9 (VBUS)
- net VCC: now also U2.5 (VBUS), J3.1 (Pin_1)
- net at D42.2 (A), MX42.1: now also MX74.2
- net at D59.2 (A), MX59.1: now also MX62.1
- net at MX17.2, MX3.2, MX31.2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: now also MX62.2
- net at D57.2 (A), MX57.1: now also MX60.1
- net at D68.2 (A): now also MX80.1; no longer MX68.1
- net at D70.2 (A), MX70.1: now also MX78.1, MX82.2
- net at D29.2 (A), MX29.1: now also MX72.2
- net at D67.2 (A): now also MX68.1, MX66.1, MX79.1; no longer MX67.1
- net at D64.2 (A), MX64.1: now also MX63.1
- new net: D60.2 (A), MX65.1, MX67.1
Other:
- moved on the sheet: C1, C10, C11, C12, C13, C14, C15, C16, C17, C2, C3, C4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

Commit message: Pre final routing
Connections:
- net ROW1: now reaches D15.1 (K), D16.1 (K), D17.1 (K), D18.1 (K), D19.1 (K), D20.1 (K), D21.1 (K), D22.1 (K), D23.1 (K), D24.1 (K), D25.1 (K), D26.1 (K), D27.1 (K), D28.1 (K)
- net ROW2: now reaches D29.1 (K), D30.1 (K), D31.1 (K), D32.1 (K), D33.1 (K), D34.1 (K), D35.1 (K), D36.1 (K), D37.1 (K), D38.1 (K), D39.1 (K), D40.1 (K), D41.1 (K), D42.1 (K)
- net COL11: now reaches MX12.2, MX26.2, MX40.2, MX54.2, MX80.2, MX83.1
- net ROW3: now reaches D43.1 (K), D44.1 (K), D45.1 (K), D46.1 (K), D47.1 (K), D48.1 (K), D49.1 (K), D50.1 (K), D51.1 (K), D52.1 (K), D53.1 (K), D54.1 (K), D55.1 (K), D56.1 (K)
- net COL13: now reaches MX14.2, MX28.2, MX42.2, MX56.2, MX70.2, MX71.1, MX78.2, MX82.1
- net COL13: now also MX74.2; no longer MX74.1
- net COL5: now reaches MX20.2, MX34.2, MX48.2, MX6.2
- net COL4: now reaches MX19.2, MX33.2, MX47.2, MX5.2
- net ROW0: now reaches D1.1 (K), D10.1 (K), D11.1 (K), D12.1 (K), D13.1 (K), D14.1 (K), D2.1 (K), D3.1 (K), D4.1 (K), D5.1 (K), D6.1 (K), D7.1 (K), D8.1 (K), D9.1 (K)
- net COL1: now reaches MX16.2, MX2.2, MX30.2, MX44.2, MX58.2, MX61.2
- net ROW4: now reaches D57.1 (K), D58.1 (K), D59.1 (K), D60.1 (K), D64.1 (K), D67.1 (K), D68.1 (K), D69.1 (K), D70.1 (K)
- net COL6: now reaches MX21.2, MX35.2, MX49.2, MX7.2
- net COL9: now reaches MX10.2, MX24.2, MX38.2, MX52.2, MX65.2, MX67.2
- net COL12: now reaches MX13.2, MX27.2, MX41.2, MX55.2, MX69.2, MX73.2, MX76.1, MX77.2, MX81.1, MX84.1
- net COL10: now reaches MX11.2, MX25.2, MX39.2, MX53.2, MX79.2
- net COL10: now also MX66.1, MX68.1; no longer MX66.2, MX68.2
- net COL8: now reaches MX23.2, MX37.2, MX51.2, MX9.2
- net COL7: now reaches MX22.2, MX36.2, MX50.2, MX63.2, MX64.2, MX8.2
- net COL0: now reaches MX1.2, MX15.2, MX29.2, MX43.2, MX57.2, MX60.2, MX72.1, MX75.2
- net at D67.2 (A), MX79.1: now also MX66.2, MX68.2; no longer MX66.1, MX68.1
- net at D42.2 (A), MX42.1: now also MX74.1; no longer MX74.2
- net COL2: now reaches MX17.2, MX3.2, MX31.2, MX45.2, MX59.2, MX62.2
- net COL3: now reaches MX18.2, MX32.2, MX4.2, MX46.2
Other:
- moved on the sheet: MX66, MX68, MX74
